File: SurfaceEEG_V1.4.brd (EAGLE design)
At the start: 41.2 x 35.5 mm, 71 parts, among them IC1 LMV602, IC2 TSZ124IQ4T, U1 MCP4442-103E/ST, U2 ATMEGA328P-MU, U3 NRF24L01ALT1

Commit message: Added active ground
Ku = 50 dB on 50 Hz
A low-pass filter = -6 dB/octave, 1 kHz = 26 dB, 22 kHz = 0 dB
Parts:
- added ACTIVE_GND: (no value), SparkFun-Connectors:1X01
- added C3: 2.2nF, (manufact)-Kemet-element14:CAPC1005X60N
- added R22: 3.3K Ohms, (manufact)-resistors-YAGEO-element14:RESC1608X60N
- added R23: 1.5M Ohms, (manufact)-resistors-YAGEO-element14:RESC1608X60N
- added R24: 220K Ohms, (manufact)-resistors-YAGEO-element14:RESC1608X60N
Connections:
- new net N$10: ACTIVE_GND.1, R24.1
- new net N$3: C3.2, IC1.6, R22.2, R23.1
- new net N$6: C3.1, IC1.7, R23.2, R24.2
- net CH0: now also R22.1
- net GNDI: now also IC1.5
Changed lines of the file:
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@@
 <attribute name="MPN" value="RT0603FRE0782KL" x="30.4" y="6.3" size="1.778" layer="27" rot="R270" display="off"/>
 </element>
+<element name="R22" library="(manufact)-resistors-YAGEO-element14" package="RESC1608X60N" value="3.3K Ohms" x="-4.9" y="-19.4">
+<attribute name="OC_FARNELL" value="1117258" x="-4.9" y="-19.4" size="1.778" layer="27" display="off"/>
+<attribute name="TOLERANCE" value="±1%" x="-4.9" y="-19.4" size="1.778" layer="27" display="off"/>
+<attribute name="WATTAGE" value="1/10 W" x="-4.9" y="-19.4" size="1.778" layer="27" display="off"/>
+<attribute name="OC_NEWARK" value="68R0079" x="-4.9" y="-19.4" size="1.778" layer="27" display="off"/>
+<attribute name="MPN" value="RC0603FR-073K3L" x="-4.9" y="-19.4" size="1.778" layer="27" display="off"/>
+<attribute name="SUPPLIER" value="Yageo" x="-4.9" y="-19.4" size="1.778" layer="27" display="off"/>
+</element>
+<element name="R23" library="(manufact)-resistors-YAGEO-element14" package="RESC1608X60N" value="1.5M Ohms" x="-4.9" y="-27.4">
+<attribute name="OC_FARNELL" value="1117246" x="-4.9" y="-27.4" size="1.778" layer="27" display="off"/>
+<attribute name="TOLERANCE" value="±1%" x="-4.9" y="-27.4" size="1.778" layer="27" display="off"/>
+<attribute name="WATTAGE" value="1/10 W" x="-4.9" y="-27.4" size="1.778" layer="27" display="off"/>
+<attribute name="OC_NEWARK" value="98K7362" x="-4.9" y="-27.4" size="1.778" layer="27" display="off"/>
+<attribute name="MPN" value="RC0603FR-071M5L" x="-4.9" y="-27.4" size="1.778" layer="27" display="off"/>
+<attribute name="SUPPLIER" value="Yageo" x="-4.9" y="-27.4" size="1.778" layer="27" display="off"/>
+</element>
+<element name="R24" library="(manufact)-resistors-YAGEO-element14" package="RESC1608X60N" value="220K Ohms" x="-4.9" y="-35.4">
+<attribute name="OC_FARNELL" value="1117252" x="-4.9" y="-35.4" size="1.778" layer="27" display="off"/>
+<attribute name="TOLERANCE" value="±1%" x="-4.9" y="-35.4" size="1.778" layer="27" display="off"/>
+<attribute name="WATTAGE" value="1/10 W" x="-4.9" y="-35.4" size="1.778" layer="27" display="off"/>
+<attribute name="OC_NEWARK" value="68R0074" x="-4.9" y="-35.4" size="1.778" layer="27" display="off"/>
+<attribute name="MPN" value="RC0603FR-07220KL" x="-4.9" y="-35.4" size="1.778" layer="27" display="off"/>
+<attribute name="SUPPLIER" value="Yageo" x="-4.9" y="-35.4" size="1.778" layer="27" display="off"/>
+</element>
+<element name="C3" library="(manufact)-Kemet-element14" package="CAPC1005X60N" value="2.2nF" x="-4.9" y="-43.4">
+<attribute name="OC_FARNELL" value="1414582" x="-4.9" y="-43.4" size="1.778" layer="27" display="off"/>
+<attribute name="TOLERANCE" value="±10%" x="-4.9" y="-43.4" size="1.778" layer="27" display="off"/>
+<attribute name="OC_NEWARK" value="70K9080" x="-4.9" y="-43.4" size="1.778" layer="27" display="off"/>
+<attribute name="VOLTAGERATING" value="50V" x="-4.9" y="-43.4" size="1.778" layer="27" display="off"/>
+<attribute name="MPN" value="C0402C222K5RACTU" x="-4.9" y="-43.4" size="1.778" layer="27" display="off"/>
+<attribute name="SUPPLIER" value="Kemet" x="-4.9" y="-43.4" size="1.778" layer="27" display="off"/>
+</element>
+<element name="ACTIVE_GND" library="SparkFun-Connectors" package="1X01" value="" x="0.4" y="-56.7"/>
 </elements>
 <signals>
@@
 <wire x1="11.4618" y1="25.5" x2="11.4618" y2="23.7" width="0.254" layer="1"/>
 <wire x1="11.4618" y1="23.7" x2="11.0618" y2="23.3" width="0.254" layer="1"/>
+<contactref element="IC1" pad="5"/>
+<wire x1="30.8" y1="26.5" x2="34.675" y2="26" width="0" layer="19" extent="1-1"/>
 </signal>
 <signal name="N$18">
@@
 <wire x1="25.0618" y1="32.6" x2="22.9538" y2="32.6" width="0.254" layer="1"/>
 <wire x1="22.9538" y1="32.6" x2="22.5" y2="32.1462" width="0.254" layer="1"/>
+<contactref element="R22" pad="1"/>
+<wire x1="-5.7382" y1="-19.4" x2="22.5" y2="32.1462" width="0" layer="19" extent="1-1"/>
 </signal>
 <signal name="N$4">
@@
 <wire x1="2.4" y1="20.362" x2="2.5" y2="20.262" width="0.254" layer="1"/>
 </signal>
+<signal name="N$3">
+<contactref element="IC1" pad="6"/>
+<contactref element="R22" pad="2"/>
+<contactref element="R23" pad="1"/>
+<contactref element="C3" pad="2"/>
+<wire x1="-4.0618" y1="-19.4" x2="34.025" y2="26" width="0" layer="19" extent="1-1"/>
+<wire x1="-5.7382" y1="-27.4" x2="-4.0618" y2="-19.4" width="0" layer="19" extent="1-1"/>
+<wire x1="-4.4174" y1="-43.4" x2="-5.7382" y2="-27.4" width="0" layer="19" extent="1-1"/>
+</signal>
+<signal name="N$6">
+<contactref element="IC1" pad="7"/>
+<contactref element="R23" pad="2"/>
+<contactref element="R24" pad="2"/>
+<contactref element="C3" pad="1"/>
+<wire x1="-4.0618" y1="-27.4" x2="33.375" y2="26" width="0" layer="19" extent="1-1"/>
+<wire x1="-4.0618" y1="-35.4" x2="-4.0618" y2="-27.4" width="0" layer="19" extent="1-1"/>
+<wire x1="-5.3826" y1="-43.4" x2="-4.0618" y2="-35.4" width="0" layer="19" extent="1-1"/>
+</signal>
+<signal name="N$10">
+<contactref element="R24" pad="1"/>
+<contactref element="ACTIVE_GND" pad="1"/>
+<wire x1="-5.7382" y1="-35.4" x2="0.4" y2="-56.7" width="0" layer="19" extent="1-1"/>
+</signal>
 </signals>
