File: SurfaceEEG_V1.4.brd (EAGLE design)
At the start: 41.2 x 35.5 mm, 76 parts, among them IC1 LMV602, IC2 TSZ124IQ4T, U1 MCP4442-103E/ST, U2 ATMEGA328P-MU, U3 NRF24L01ALT1

Commit message: Module active ground completed
Parts:
- removed ACTIVE_GND: (no value), SparkFun-Connectors:1X01
- added J1: (no value), SparkFun-Connectors:PAD-1.5X4.5
- moved C3 74.7 mm to (30.7, 22.3)
- moved R24 66.8 mm to (33.4, 19.3), turned to 180 degrees
- moved R23 62.2 mm to (30.6, 23.7), turned to 180 degrees
- moved R22 53.4 mm to (31.2, 20.0), turned to 90 degrees
- moved C1 0.58 mm to (35.2, 27.7)
- moved R2 0.20 mm to (36.0, 20.9)
Connections:
- net CH0: no longer R22.1
- net CH0_F_A: now also R22.1
- net N$10: now also J1.P$1; no longer ACTIVE_GND.1
Routing:
- net N$6: track 0.00 -> 11.4 mm
- net CH0_F_A: track 26.8 -> 36.3 mm
- net N$3: track 0.00 -> 7.32 mm
- net N$10: track 0.00 -> 4.21 mm
- net GNDI: track 111.8 -> 115.8 mm
- net VDD: track 88.1 -> 87.2 mm
- net CH0_F: track 25.7 -> 26.4 mm

Commit message: Board changed after library changes
After making fonts smaller, the board have changed
Parts:
- R19, R20: value 88.7K EDIT -> 82K Ohms
