File: SurfaceEEG_V1.4.sch (EAGLE design)
At the start: 67 parts, among them IC1 LMV602, IC2 TSZ124IQ4T, U1 MCP4442-103E/ST

Commit message: Started version 1.4 with atmega328
Parts:
- removed R11, R16: 3.3K Ohms, (manufact)-resistors-YAGEO-element14:RC0603FR-073K3L
- added R13, R21: 4.7K Ohms, (manufact)-resistors-YAGEO-element14:9C04021A4701JLHF3
- added U$7: NRF24L01SMD, (misc)-parts-that-we-use:NRF24L01SMD
- added U2: ATMEGA328P-MU, (misc)-parts-that-we-use:ATMEGA328P-MU
Connections:
- net SCL: now also R13.R1; no longer R16.R1
- net SDA: now also R21.R2; no longer R11.R2
- net VCC: now also R13.R2, R21.R1; no longer R11.R1, R16.R2
Changed lines of the file:
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@@
 <grid distance="0.1" unitdist="inch" unit="inch" style="lines" multiple="1" display="no" altdistance="0.01" altunitdist="inch" altunit="inch"/>
 <layers>
-<layer number="1" name="Top" color="4" fill="1" visible="yes" active="no"/>
-<layer number="2" name="Route2" color="1" fill="3" visible="yes" active="no"/>
-<layer number="3" name="Route3" color="4" fill="3" visible="yes" active="no"/>
-<layer number="14" name="Route14" color="1" fill="6" visible="yes" active="no"/>
-<layer number="15" name="Route15" color="4" fill="6" visible="yes" active="no"/>
-<layer number="16" name="Bottom" color="1" fill="1" visible="yes" active="no"/>
-<layer number="17" name="Pads" color="2" fill="1" visible="yes" active="no"/>
-<layer number="18" name="Vias" color="2" fill="1" visible="yes" active="no"/>
-<layer number="19" name="Unrouted" color="6" fill="1" visible="yes" active="no"/>
-<layer number="20" name="Dimension" color="15" fill="1" visible="yes" active="no"/>
-<layer number="21" name="tPlace" color="7" fill="1" visible="yes" active="no"/>
-<layer number="22" name="bPlace" color="7" fill="1" visible="yes" active="no"/>
-<layer number="23" name="tOrigins" color="15" fill="1" visible="yes" active="no"/>
-<layer number="24" name="bOrigins" color="15" fill="1" visible="yes" active="no"/>
-<layer number="25" name="tNames" color="7" fill="1" visible="yes" active="no"/>
-<layer number="26" name="bNames" color="7" fill="1" visible="yes" active="no"/>
-<layer number="27" name="tValues" color="7" fill="1" visible="yes" active="no"/>
-<layer number="28" name="bValues" color="7" fill="1" visible="yes" active="no"/>
+<layer number="1" name="Top" color="4" fill="1" visible="no" active="no"/>
+<layer number="2" name="Route2" color="1" fill="3" visible="no" active="no"/>
+<layer number="3" name="Route3" color="4" fill="3" visible="no" active="no"/>
+<layer number="14" name="Route14" color="1" fill="6" visible="no" active="no"/>
+<layer number="15" name="Route15" color="4" fill="6" visible="no" active="no"/>
+<layer number="16" name="Bottom" color="1" fill="1" visible="no" active="no"/>
+<layer number="17" name="Pads" color="2" fill="1" visible="no" active="no"/>
+<layer number="18" name="Vias" color="2" fill="1" visible="no" active="no"/>
+<layer number="19" name="Unrouted" color="6" fill="1" visible="no" active="no"/>
+<layer number="20" name="Dimension" color="15" fill="1" visible="no" active="no"/>
+<layer number="21" name="tPlace" color="7" fill="1" visible="no" active="no"/>
+<layer number="22" name="bPlace" color="7" fill="1" visible="no" active="no"/>
+<layer number="23" name="tOrigins" color="15" fill="1" visible="no" active="no"/>
+<layer number="24" name="bOrigins" color="15" fill="1" visible="no" active="no"/>
+<layer number="25" name="tNames" color="7" fill="1" visible="no" active="no"/>
+<layer number="26" name="bNames" color="7" fill="1" visible="no" active="no"/>
+<layer number="27" name="tValues" color="7" fill="1" visible="no" active="no"/>
+<layer number="28" name="bValues" color="7" fill="1" visible="no" active="no"/>
 <layer number="29" name="tStop" color="7" fill="3" visible="no" active="no"/>
 <layer number="30" name="bStop" color="7" fill="6" visible="no" active="no"/>
@@
 <layer number="35" name="tGlue" color="7" fill="4" visible="no" active="no"/>
 <layer number="36" name="bGlue" color="7" fill="5" visible="no" active="no"/>
-<layer number="37" name="tTest" color="7" fill="1" visible="yes" active="no"/>
-<layer number="38" name="bTest" color="7" fill="1" visible="yes" active="no"/>
+<layer number="37" name="tTest" color="7" fill="1" visible="no" active="no"/>
+<layer number="38" name="bTest" color="7" fill="1" visible="no" active="no"/>
 <layer number="39" name="tKeepout" color="4" fill="11" visible="no" active="no"/>
 <layer number="40" name="bKeepout" color="1" fill="11" visible="no" active="no"/>
@@
 <layer number="44" name="Drills" color="7" fill="1" visible="no" active="no"/>
 <layer number="45" name="Holes" color="7" fill="1" visible="no" active="no"/>
-<layer number="46" name="Milling" color="3" fill="1" visible="yes" active="no"/>
-<layer number="47" name="Measures" color="7" fill="1" visible="yes" active="no"/>
-<layer number="48" name="Document" color="7" fill="1" visible="yes" active="no"/>
-<layer number="49" name="Reference" color="7" fill="1" visible="yes" active="no"/>
-<layer number="50" name="dxf" color="7" fill="1" visible="yes" active="no"/>
-<layer number="51" name="tDocu" color="7" fill="1" visible="yes" active="no"/>
-<layer number="52" name="bDocu" color="7" fill="1" visible="yes" active="no"/>
-<layer number="53" name="tGND_GNDA" color="7" fill="9" visible="yes" active="no"/>
-<layer number="54" name="bGND_GNDA" color="1" fill="9" visible="yes" active="no"/>
-<layer number="56" name="wert" color="7" fill="1" visible="yes" active="no"/>
-<layer number="57" name="tCAD" color="7" fill="1" visible="yes" active="no"/>
-<layer number="58" name="bCopper" color="7" fill="1" visible="yes" active="no"/>
-<layer number="59" name="tCarbon" color="7" fill="1" visible="yes" active="no"/>
-<layer number="60" name="bCarbon" color="7" fill="1" visible="yes" active="no"/>
-<layer number="61" name="stand" color="7" fill="1" visible="yes" active="no"/>
+<layer number="46" name="Milling" color="3" fill="1" visible="no" active="no"/>
+<layer number="47" name="Measures" color="7" fill="1" visible="no" active="no"/>
+<layer number="48" name="Document" color="7" fill="1" visible="no" active="no"/>
+<layer number="49" name="Reference" color="7" fill="1" visible="no" active="no"/>
+<layer number="50" name="dxf" color="7" fill="1" visible="no" active="no"/>
+<layer number="51" name="tDocu" color="7" fill="1" visible="no" active="no"/>
+<layer number="52" name="bDocu" color="7" fill="1" visible="no" active="no"/>
+<layer number="53" name="tGND_GNDA" color="7" fill="9" visible="no" active="no"/>
+<layer number="54" name="bGND_GNDA" color="1" fill="9" visible="no" active="no"/>
+<layer number="56" name="wert" color="7" fill="1" visible="no" active="no"/>
+<layer number="57" name="tCAD" color="7" fill="1" visible="no" active="no"/>
+<layer number="58" name="bCopper" color="7" fill="1" visible="no" active="no"/>
+<layer number="59" name="tCarbon" color="7" fill="1" visible="no" active="no"/>
+<layer number="60" name="bCarbon" color="7" fill="1" visible="no" active="no"/>
+<layer number="61" name="stand" color="7" fill="1" visible="no" active="no"/>
 <layer number="90" name="Modules" color="5" fill="1" visible="yes" active="yes"/>
 <layer number="91" name="Nets" color="2" fill="1" visible="yes" active="yes"/>
@@
 <part name="R14" library="(manufact)-resistors-YAGEO-element14" deviceset="RC0603FR-073K3L" device="" value="3.3K Ohms"/>
 <part name="R15" library="(manufact)-resistors-YAGEO-element14" deviceset="RC0603FR-073K3L" device="" value="3.3K Ohms"/>
-<part name="R16" library="(manufact)-resistors-YAGEO-element14" deviceset="RC0603FR-073K3L" device="" value="3.3K Ohms"/>
-<part name="R11" library="(manufact)-resistors-YAGEO-element14" deviceset="RC0603FR-073K3L" device="" value="3.3K Ohms"/>
 <part name="R17" library="(manufact)-resistors-YAGEO-element14" deviceset="RC0603FR-07220KL" device="" value="220K Ohms"/>
 <part name="R3" library="(manufact)-resistors-YAGEO-element14" deviceset="RC0603FR-07220KL" device="" value="220K Ohms"/>
@@
 <part name="PH4" library="(misc)-parts-that-we-use" deviceset="PH1X3" device=""/>
 <part name="U$6" library="(misc)-parts-that-we-use" deviceset="NRF24LE1-24" device=""/>
+<part name="R13" library="(manufact)-resistors-YAGEO-element14" deviceset="9C04021A4701JLHF3" device="" value="4.7K Ohms"/>
+<part name="R21" library="(manufact)-resistors-YAGEO-element14" deviceset="9C04021A4701JLHF3" device="" value="4.7K Ohms"/>
+<part name="U$7" library="(misc)-parts-that-we-use" deviceset="NRF24L01" device="SMD"/>
+<part name="U2" library="(misc)-parts-that-we-use" deviceset="ATMEGA328P-MU" device=""/>
 </parts>
 <sheets>
@@
 <instance part="R14" gate="A" x="-60.96" y="116.84"/>
 <instance part="R15" gate="A" x="-60.96" y="101.6"/>
-<instance part="R16" gate="A" x="-83.82" y="53.34"/>
-<instance part="R11" gate="A" x="-20.32" y="55.88"/>
 <instance part="R17" gate="A" x="-104.14" y="147.32" rot="R90"/>
 <instance part="R3" gate="A" x="-104.14" y="127" rot="R90"/>
@@
 <instance part="PH4" gate="G$1" x="-22.86" y="190.5"/>
 <instance part="U$6" gate="G$1" x="203.2" y="104.14"/>
+<instance part="R13" gate="A" x="-83.82" y="53.34"/>
+<instance part="R21" gate="A" x="-20.32" y="55.88"/>
+<instance part="U$7" gate="G$1" x="162.56" y="165.1"/>
+<instance part="U2" gate="A" x="266.7" y="27.94"/>
 </instances>
 <busses>
@@
 </segment>
 <segment>
+<pinref part="P+9" gate="VCC" pin="VCC"/>
+<pinref part="R21" gate="A" pin="R1"/>
+</segment>
+<segment>
 <pinref part="P+8" gate="VCC" pin="VCC"/>
-<pinref part="R16" gate="A" pin="R2"/>
-</segment>
-<segment>
-<pinref part="R11" gate="A" pin="R1"/>
-<pinref part="P+9" gate="VCC" pin="VCC"/>
+<pinref part="R13" gate="A" pin="R2"/>
 </segment>
 </net>
@@
 <wire x1="-63.5" y1="53.34" x2="-71.12" y2="53.34" width="0.1524" layer="91"/>
 <label x="-71.12" y="53.34" size="1.778" layer="95"/>
-<pinref part="R16" gate="A" pin="R1"/>
+<pinref part="R13" gate="A" pin="R1"/>
 </segment>
 <segment>
@@
 <wire x1="-27.94" y1="55.88" x2="-20.32" y2="55.88" width="0.1524" layer="91"/>
 <label x="-25.4" y="55.88" size="1.778" layer="95"/>
-<pinref part="R11" gate="A" pin="R2"/>
-</segment>
-<segment>
+<pinref part="R21" gate="A" pin="R2"/>
+</segment>
+<segment>
