File: SurfaceEEG_Central_V1.0.sch (EAGLE design)
At the start: 18 parts, among them IC1 LMV602

Commit message: Central unit completed, testing module added
Parts:
- added C10, C25: 10uF, (manufact)-Kemet-element14:C0603C106M9PACTU
- added C11: 100uF, (manufact)-Kemet-element14:C1206C107M9PACTU
- added C12, C13, C14, C15: 100nF, (manufact)-capacitors-AVX-element14:06035C104KAT2A
- added C16, C22: 1.5pF, (manufact)-capacitors-AVX-element14:UQCL2A1R5BAT2A/500
- added C17, C26: 1pF, (manufact)-capacitors-AVX-element14:UQCL2A1R0BAT2A/500
- added C18, C19, C29, C30, C8, C9: 15pF, (manufact)-capacitors-AVX-element14:UQCL2A150JAT2A/500
- added C20, C31: 47nF, (manufact)-Kemet-element14:C0603C473K1RACTU
- added C21, C32: 0.1uF, (manufact)-capacitors-AVX-element14:04023C104KAT2A
- added C23, C33: 2.2nF, (manufact)-Kemet-element14:C0402C222K5RACTU
- added C24, C34: 4.7pF, (manufact)-capacitors-AVX-element14:UQCL2A4R7CAT2A/500
- added C27, C28: 50PF, (manufact)-capacitors-AVX-element14:06035A500JAT2A
- added C35, C36: 4.7uF, (manufact)-capacitors-AVX-element14:0805YC475KAT2A
- added D2: GREEN-0603, Seeed-OPL-Diode:SMD-LED-CLEAR-GREEN(0603)
- added J1: (no value), SparkFun-Connectors:M02PTH
- added J2: (no value), SparkFun-Connectors:M01SMD-4.5X1.5
- added J3: MICRO-USB, (misc)-parts-that-we-use:MICRO-USB
- added L1, L5: 2.7nH, (manufact)-inductors-WE-KI-element14:WE-KI-744765027A_0402A
- added L2, L4: 3.9nH, (manufact)-inductors-WE-KI-element14:WE-KI-744765039A_0402A
- added L3, L6: 8.2nH, (manufact)-inductors-WE-KI-element14:WE-KI-744765082A_0402A
- added R10, R11, R13, R14: 22K Ohms, (manufact)-resistors-YAGEO-element14:RC0603FR-0722KL
- added R12, R15: 1.5K Ohms, (manufact)-resistors-YAGEO-element14:RC0603FR-071K5L
- added R16, R17: 22 Ohm, (manufact)-resistors-YAGEO-element14:9C06031A22R0JLHFT
- added R18: 2.7K Ohms, (manufact)-resistors-YAGEO-element14:RC0603FR-072K7L
- added R19: 1K Ohm, (manufact)-resistors-YAGEO-element14:9C06031A1001JLHFT
- added U$1: NCP103, (custom)-new-components:NCP103
- added U$2: RGB-LED, (custom)-new-components:RGB-LED
- added U$3: MCP73831T-2ACI/OT, (custom)-new-components:MCP73831T-2ACI/OT
- added U$4: VCC, (custom)-new-components:VCC
- added U$5: GND, (custom)-new-components:GND
- added U$6: ANTENNA_1LEFT, ant-planar-1:ANTENNA_1LEFT
- added U$7: ANTENNA_1RIGHT, ant-planar-1:ANTENNA_1RIGHT
- added U1: STM32L151CBT6, (misc)-parts-that-we-use:STM32L151CBT6
- added U2, U3: NRF24L01ALT1, Testing:NRF24L01ALT1
- added U4: HC_05, HC_08:HC_05
- added XTAL1, XTAL2, XTAL3: 7M-16.000MAAJ-T, (misc)-parts-that-we-use:7M-16.000MAAJ-T
Connections:
- removed net +3V3: C6.C2, IC1G$3.VCC+
- removed net DAC: R2.R2
- removed net NEG_VOLT_GEN: R5.R2
- new net ANT: C22.C2, C26.C2, U$6.RF
- new net ANT1: L1.1, L3.1, U3.ANT1
- new net ANT2: L2.1, L3.2, U3.ANT2
- new net ANT3: L4.1, L6.2, U2.ANT2
- new net ANT4: L5.1, L6.1, U2.ANT1
- new net BT_KEY: U1.PA7, U4.PIO3
- new net BT_LED: U1.PB0, U4.PIO1
- new net DAC_OUT: R2.R2, U1.PA4
- new net GND: C10.C1, C11.C1, C12.C1, C13.C1, C14.C1, C15.C1, C17.C1, C18.C2, C19.C2, C2.C1, C20.C1, C21.C1, C23.C1, C24.C1, C25.C1, C26.C1, C27.C2, C28.C1, C29.C2, C30.C2, C31.C1, C32.C1, C33.C1, C34.C1, C36.C1, C5.C1, C6.C1, C7.C1, C8.C2, C9.C2, D1.C2, J3.GND, R11.R2, R13.R2, R14.R2, R4.R2, R7.R2, R8.R2, U$1.GND, U$5.P$1, U$6.GND, U$7.GND, U1.VSSA, U1.VSS_1, U1.VSS_2, U1.VSS_3, U2.VSS@0, U2.VSS@14, U2.VSS@17, U2.VSS@20, U2.VSS@8, U3.VSS@0, U3.VSS@14, U3.VSS@17, U3.VSS@20, U3.VSS@8, U4.GND
- new net MISO: U1.PB14, U2.MISO, U3.MISO
- new net MOSI: U1.PB15, U2.MOSI, U3.MOSI
- new net N$10: C29.C1, U3.XC1, XTAL3.3
- new net N$11: R10.R1, U$1.EN
- new net N$12: C30.C1, U3.XC2, XTAL3.1
- new net N$13: C22.C1, L2.2
- new net N$14: C8.C1, U1.PH1-OSC_OUT, XTAL1.3
- new net N$15: C9.C1, U1.PH0-OSC_IN, XTAL1.1
- new net N$16: C33.C2, C34.C2, L1.2, U3.VDD_PA
- new net N$17: U$2.R, U1.PA2
- new net N$18: U$2.B, U1.PA3
- new net N$19: R11.R1, U3.IREF
- new net N$20: C31.C2, U3.DVDD
- new net N$21: U$2.G, U1.PA1
- new net N$22: R12.R1, U$2.COM
- new net N$23: J1.1, R13.R1, U1.BOOT0
- new net N$24: C18.C1, U2.XC1, XTAL2.3
- new net N$25: C23.C2, C24.C2, L5.2, U2.VDD_PA
- new net N$26: R14.R1, U2.IREF
- new net N$27: C20.C2, U2.DVDD
- new net N$28: C16.C1, L4.2
- new net N$29: C19.C1, U2.XC2, XTAL2.1
- new net N$30: C16.C2, C17.C2, U$7.RF
- new net N$31: C35.C2, D2.+, J3.VBUS, U$3.VDD
- new net N$32: C28.C2, J3.D+, R15.R1, R17.R2
- new net N$33: C27.C1, J3.D-, R16.R2
- new net N$34: R18.R1, U$3.PROG
- new net N$36: D2.-, R19.R1
- new net N$37: R19.R2, U$3.STAT
- new net PWM_GEN: R5.R2, U1.PA6
- new net RCV_CE: U1.PB11, U3.CE
- new net RCV_CS: U1.PB10, U3.CSN
- new net SCLK: U1.PB13, U2.SCK, U3.SCK
- new net TRN_CE: U1.PB6, U2.CE
- new net TRN_CS: U1.PB5, U2.CSN
- new net UART1_RX: U1.PA10, U4.TX
- new net UART1_TX: U1.PA9, U4.RX
- new net USB_DM: R16.R1, U1.PA11
- new net USB_DP: R17.R1, U1.PA12
- new net VBAT: C10.C2, C36.C2, R10.R2, U$1.IN, U$3.VBAT, U$4.P$1
- new net VCC: C11.C2, C12.C2, C13.C2, C14.C2, C15.C2, C21.C2, C25.C2, C32.C2, C6.C2, IC1G$3.VCC+, J1.2, R12.R2, R15.R2, U$1.OUT, U1.VDDA, U1.VDD_1, U1.VDD_2, U1.VDD_3, U2.VDD@15, U2.VDD@18, U2.VDD@7, U3.VDD@15, U3.VDD@18, U3.VDD@7, U4.3V3
- net 0V: now also C35.C1, R18.R2, U$3.VSS; no longer C2.C1, C5.C1, C6.C1, C7.C1, D1.C2, R4.R2, R7.R2, R8.R2
- net ACTIVE_GND: now also J2.1
Other:
- note added: "NRF supply VCC"
